Commit message: 更新了机械臂模型，增加了夹爪和桌子方块场景

File: TG_Robot/src/robot_gazebo/config/gazebo_arm620_lerobot.urdf.xacro (robot description, xacro)
@@ -33,8 +33,208 @@
         <gravity>false</gravity>
     </gazebo>
+    <gazebo reference="gripper_base">
+        <material>Gazebo/Black</material>
+        <gravity>false</gravity>
+    </gazebo>
+    <gazebo reference="hand_narrow1_Link">
+        <material>Gazebo/DarkGrey</material>
+        <gravity>false</gravity>
+    </gazebo>
+    <gazebo reference="hand_narrow2_Link">
+        <material>Gazebo/DarkGrey</material>
+        <gravity>false</gravity>
+    </gazebo>
+    <gazebo reference="hand_narrow3_Link">
+        <material>Gazebo/DarkGrey</material>
+        <gravity>false</gravity>
+    </gazebo>
+    <gazebo reference="hand_wide1_Link">
+        <material>Gazebo/DarkGrey</material>
+        <gravity>false</gravity>
+    </gazebo>
+    <gazebo reference="hand_wide2_Link">
+        <material>Gazebo/DarkGrey</material>
+        <gravity>false</gravity>
+    </gazebo>
+    <gazebo reference="hand_wide3_Link">
+        <material>Gazebo/DarkGrey</material>
+        <gravity>false</gravity>
+    </gazebo>
+    <gazebo reference="hand_narrow_loop_Link">
+        <material>Gazebo/DarkGrey</material>
+        <mu1>1.6</mu1>
+        <mu2>1.6</mu2>
+        <kp>1000000.0</kp>
+        <kd>5.0</kd>
+    </gazebo>
+    <gazebo reference="hand_wide_loop_Link">
+        <material>Gazebo/DarkGrey</material>
+        <mu1>1.6</mu1>
+        <mu2>1.6</mu2>
+        <kp>1000000.0</kp>
+        <kd>5.0</kd>
+    </gazebo>
     <gazebo>
         <is_static>false</is_static>
         <self_collide>false</self_collide>
     </gazebo>
+    <!-- OmniPicker gripper: simplified bilateral linkage for stable grasping -->
+    <joint name="gripper_base_joint" type="fixed">
+        <origin xyz="0 0 0.022" rpy="0 0 1.5708"/>
+        <parent link="Link6"/>
+        <child link="gripper_base"/>
+    </joint>
+    <link name="gripper_base">
+        <inertial>
+            <origin xyz="-0.00005520 1.2341E-05 0.03296193" rpy="0 0 0"/>
+            <mass value="0.25641368"/>
+            <inertia ixx="4.6351E-04" ixy="-1.0E-08" ixz="-1.04E-06" iyy="4.4525E-04" iyz="-5.00E-08" izz="1.0438E-04"/>
+        </inertial>
+        <visual>
+            <origin xyz="0 0 0" rpy="0 0 0"/>
+            <geometry>
+                <mesh filename="file://$(find robot_description)/meshes/omnipicker_gripper/base_link.STL"/>
+            </geometry>
+        </visual>
+        <collision>
+            <origin xyz="0 0 0" rpy="0 0 0"/>
+            <geometry>
+                <mesh filename="file://$(find robot_description)/meshes/omnipicker_gripper/base_link.STL"/>
+            </geometry>
+        </collision>
+    </link>
+    <!-- Visual follower links: rigidly attach full OmniPicker geometry to each driven finger -->
+    <link name="hand_narrow1_Link">
+        <visual>
+            <origin xyz="0 0 0" rpy="0 0 0"/>
+            <geometry>
+                <mesh filename="file://$(find robot_description)/meshes/omnipicker_gripper/narrow1_Link.STL"/>
+            </geometry>
+        </visual>
+    </link>
+    <joint name="hand_narrow1_joint" type="fixed">
+        <origin xyz="-0.01737 -0.002133 -0.000028" rpy="0 0 0"/>
+        <parent link="hand_narrow_loop_Link"/>
+        <child link="hand_narrow1_Link"/>
+    </joint>
+    <link name="hand_narrow2_Link">
+        <visual>
+            <origin xyz="0 0 0" rpy="0 0 0"/>
+            <geometry>
+                <mesh filename="file://$(find robot_description)/meshes/omnipicker_gripper/narrow2_Link.STL"/>
+            </geometry>
+        </visual>
+    </link>
+    <joint name="hand_narrow2_joint" type="fixed">
+        <origin xyz="0.030852 0.018551 0" rpy="0 0 0"/>
+        <parent link="hand_narrow1_Link"/>
+        <child link="hand_narrow2_Link"/>
+    </joint>
+    <link name="hand_narrow3_Link">
+        <visual>
+            <origin xyz="0 0 0" rpy="0 0 0"/>
+            <geometry>
+                <mesh filename="file://$(find robot_description)/meshes/omnipicker_gripper/narrow3_Link.STL"/>
+            </geometry>
+        </visual>
+    </link>
+    <joint name="hand_narrow3_joint" type="fixed">
+        <origin xyz="0.018118 -0.01574 0" rpy="0 0 0"/>
+        <parent link="hand_narrow2_Link"/>
+        <child link="hand_narrow3_Link"/>
+    </joint>
+    <link name="hand_wide1_Link">
+        <visual>
+            <origin xyz="0 0 0" rpy="0 0 0"/>
+            <geometry>
+                <mesh filename="file://$(find robot_description)/meshes/omnipicker_gripper/wide1_Link.STL"/>
+            </geometry>
+        </visual>
+    </link>
+    <joint name="hand_wide1_joint" type="fixed">
+        <origin xyz="-0.01737 0.002133 0.000028" rpy="0 0 0"/>
+        <parent link="hand_wide_loop_Link"/>
+        <child link="hand_wide1_Link"/>
+    </joint>
+    <link name="hand_wide2_Link">
+        <visual>
+            <origin xyz="0 0 0" rpy="0 0 0"/>
+            <geometry>
+                <mesh filename="file://$(find robot_description)/meshes/omnipicker_gripper/wide2_Link.STL"/>
+            </geometry>
+        </visual>
+    </link>
+    <joint name="hand_wide2_joint" type="fixed">
+        <origin xyz="0.030852 -0.018551 0" rpy="0 0 0"/>
+        <parent link="hand_wide1_Link"/>
+        <child link="hand_wide2_Link"/>
+    </joint>
+    <link name="hand_wide3_Link">
+        <visual>
+            <origin xyz="0 0 0" rpy="0 0 0"/>
+            <geometry>
+                <mesh filename="file://$(find robot_description)/meshes/omnipicker_gripper/wide3_Link.STL"/>
+            </geometry>
+        </visual>
+    </link>
+    <joint name="hand_wide3_joint" type="fixed">
+        <origin xyz="0.018118 0.01574 0" rpy="0 0 0"/>
+        <parent link="hand_wide2_Link"/>
+        <child link="hand_wide3_Link"/>
+    </joint>
+    <link name="hand_narrow_loop_Link">
+        <inertial>
+            <origin xyz="0.014869 -0.0036066 0.00029307" rpy="0 0 0"/>
+            <mass value="0.022591"/>
+            <inertia ixx="4.3916E-06" ixy="1.114E-07" ixz="-4.9655E-12" iyy="4.737E-06" iyz="1.7121E-11" izz="6.0445E-07"/>
+        </inertial>
+        <visual>
+            <origin xyz="0 0 0" rpy="0 0 0"/>
+            <geometry>
+                <mesh filename="file://$(find robot_description)/meshes/omnipicker_gripper/narrow_loop_Link.STL"/>
+            </geometry>
+        </visual>
+        <collision>
+            <origin xyz="0.014 0.0 0.0" rpy="0 0 0"/>
+            <geometry>
+                <box size="0.040 0.010 0.020"/>
+            </geometry>
+        </collision>
+    </link>
+    <joint name="hand_narrow_loop_joint" type="revolute">
+        <origin xyz="0 -0.021633 0.07387" rpy="-2.9951 -1.5708 -0.15964"/>
+        <parent link="gripper_base"/>
+        <child link="hand_narrow_loop_Link"/>
+        <axis xyz="0 0 -1"/>
+        <limit lower="-1.2" upper="1.2" effort="10" velocity="4.0"/>
+        <dynamics damping="0.6" friction="0.2"/>
+    </joint>
+    <link name="hand_wide_loop_Link">
+        <inertial>
+            <origin xyz="0.016268 0.0040555 0.00030323" rpy="0 0 0"/>
+            <mass value="0.025142"/>
+            <inertia ixx="5.887E-06" ixy="-1.1234E-07" ixz="2.1954E-11" iyy="6.236E-06" iyz="-9.473E-12" izz="6.2389E-07"/>
+        </inertial>
+        <visual>
+            <origin xyz="0 0 0" rpy="0 0 0"/>
+            <geometry>
+                <mesh filename="file://$(find robot_description)/meshes/omnipicker_gripper/wide_loop_Link.STL"/>
+            </geometry>
+        </visual>
+        <collision>
+            <origin xyz="0.014 0.0 0.0" rpy="0 0 0"/>
+            <geometry>
+                <box size="0.040 0.010 0.020"/>
+            </geometry>
+        </collision>
+    </link>
+    <joint name="hand_wide_loop_joint" type="revolute">
+        <origin xyz="0 0.021633 0.07387" rpy="-2.9951 -1.5708 -0.15964"/>
+        <parent link="gripper_base"/>
+        <child link="hand_wide_loop_Link"/>
+        <axis xyz="0 0 -1"/>
+        <limit lower="-1.2" upper="1.2" effort="10" velocity="4.0"/>
+        <dynamics damping="0.6" friction="0.2"/>
+    </joint>
     <!-- Overview camera 1: front view (see full robot body) -->
     <link name="front_camera_link">
@@ -188,4 +388,18 @@
             <state_interface name="velocity"/>
         </joint>
+        <joint name="hand_narrow_loop_joint">
+            <command_interface name="position"/>
+            <state_interface name="position">
+                <param name="initial_value">0.0</param>
+            </state_interface>
+            <state_interface name="velocity"/>
+        </joint>
+        <joint name="hand_wide_loop_joint">
+            <command_interface name="position"/>
+            <state_interface name="position">
+                <param name="initial_value">0.0</param>
+            </state_interface>
+            <state_interface name="velocity"/>
+        </joint>
     </ros2_control>
     <!-- Load ros2_control plugin -->
